Commit message: Closes #2

File: tr5_basic.urdf.xacro (robot description, xacro)
@@ -5,4 +5,5 @@
     <!--<xacro:property name="pi" value="3.14159265" />-->
     <!-- @todo Inertia parameters -->
+    <xacro:property name="base_mass" value="4.0" />  <!-- CAll back function-->
     <xacro:property name="base_mass" value="4.0" />  <!-- This mass might be incorrect -->
     <xacro:property name="shoulder_mass" value="3.7000" />
